File: kicad/repl_sharp_el-w516x.sch (KiCad schematic (older format))
At the start: 29 parts, among them J1 USB_B_Micro, J2 AVR-ISP-6, SW1 SW_RESET, U1 74HC165D, U2 ATmega32U4-AU, U3 74HC595, Y1 Crystal

Commit message: kicad: fix virtual component
Parts:
- C1, C2: part_num (none) -> CC0603JRNPO9BN220
- C10, C11, C5, C9: part_num (none) -> CL10A105KP8NNNC
- C12: part_num (none) -> CL10A475KQ8NNNC
- C13, C14, C3, C4, C6, C7, C8: part_num (none) -> CL10B104KO8NNNC
- D11: part_num (none) -> SML-D12U1WT86
- DS1: part_num (none) -> NHD-C12832A1Z-FSW-FBW-3V3
- J1: part_num (none) -> 10118192-0001LF
- R1, R4: part_num (none) -> RC0603FR-0710KL
- R18: part_num (none) -> RC0603FR-071KL
- R2, R3: part_num (none) -> RC0603FR-0722RL
- SW1: part_num (none) -> PTS645SM43SMTR92 LFS
- U1: part_num (none) -> 74HC165D\\,652
- U2: part_num (none) -> ATMEGA32U4-AUR
- U3: part_num (none) -> SN74HC595DR
- Y1: part_num (none) -> ECS-80-18-30-JGN-TR
Changed lines of the file:
@@
 F 5 "1276-1005-1-ND" H 3700 5150 50  0001 C CNN "Digi-Key PN"
 F 6 "https://www.digikey.com/product-detail/en/samsung-electro-mechanics/CL10B104KO8NNNC/1276-1005-1-ND/3889091" H 3700 5150 50  0001 C CNN "Digi-Key Page"
+F 7 "CL10B104KO8NNNC" H 3700 5150 50  0001 C CNN "part_num"
 	1    3700 5150
 	0    1    -1   0
@@
 F 5 "1276-1005-1-ND" H 1750 6850 50  0001 C CNN "Digi-Key PN"
 F 6 "https://www.digikey.com/product-detail/en/samsung-electro-mechanics/CL10B104KO8NNNC/1276-1005-1-ND/3889091" H 1750 6850 50  0001 C CNN "Digi-Key Page"
+F 7 "CL10B104KO8NNNC" H 1750 6850 50  0001 C CNN "part_num"
 	1    1750 6850
 	0    -1   1    0
@@
 F 12 "NHD-C12832A1Z-FSW-FBW-3V3-ND" H 1900 6850 50  0001 C CNN "Digi-Key PN"
 F 13 "https://www.digikey.com/product-detail/en/newhaven-display-intl/NHD-C12832A1Z-FSW-FBW-3V3/NHD-C12832A1Z-FSW-FBW-3V3-ND/2059236" H 1900 6850 50  0001 C CNN "Digi-Key Page"
+F 14 "NHD-C12832A1Z-FSW-FBW-3V3" H 1900 6850 50  0001 C CNN "part_num"
 	1    1900 6850
 	1    0    0    -1
@@
 F 5 "1276-1005-1-ND" H 1450 6950 50  0001 C CNN "Digi-Key PN"
 F 6 "https://www.digikey.com/product-detail/en/samsung-electro-mechanics/CL10B104KO8NNNC/1276-1005-1-ND/3889091" H 1450 6950 50  0001 C CNN "Digi-Key Page"
+F 7 "CL10B104KO8NNNC" H 1450 6950 50  0001 C CNN "part_num"
 	1    1450 6950
 	0    -1   1    0
@@
 F 5 "1276-1005-1-ND" H 1750 7050 50  0001 C CNN "Digi-Key PN"
 F 6 "https://www.digikey.com/product-detail/en/samsung-electro-mechanics/CL10B104KO8NNNC/1276-1005-1-ND/3889091" H 1750 7050 50  0001 C CNN "Digi-Key Page"
+F 7 "CL10B104KO8NNNC" H 1750 7050 50  0001 C CNN "part_num"
 	1    1750 7050
 	0    -1   1    0
@@
 F 5 "1276-1005-1-ND" H 1450 7150 50  0001 C CNN "Digi-Key PN"
 F 6 "https://www.digikey.com/product-detail/en/samsung-electro-mechanics/CL10B104KO8NNNC/1276-1005-1-ND/3889091" H 1450 7150 50  0001 C CNN "Digi-Key Page"
+F 7 "CL10B104KO8NNNC" H 1450 7150 50  0001 C CNN "part_num"
 	1    1450 7150
 	0    -1   1    0
@@
 F 5 "1276-1005-1-ND" H 1750 7250 50  0001 C CNN "Digi-Key PN"
 F 6 "https://www.digikey.com/product-detail/en/samsung-electro-mechanics/CL10B104KO8NNNC/1276-1005-1-ND/3889091" H 1750 7250 50  0001 C CNN "Digi-Key Page"
+F 7 "CL10B104KO8NNNC" H 1750 7250 50  0001 C CNN "part_num"
 	1    1750 7250
 	0    -1   1    0
@@
 F 5 "1276-1182-1-ND" H 1750 7450 50  0001 C CNN "Digi-Key PN"
 F 6 "https://www.digikey.com/product-detail/en/samsung-electro-mechanics/CL10A105KP8NNNC/1276-1182-1-ND/3889268" H 1750 7450 50  0001 C CNN "Digi-Key Page"
+F 7 "CL10A105KP8NNNC" H 1750 7450 50  0001 C CNN "part_num"
 	1    1750 7450
 	0    -1   1    0
@@
 F 5 "1276-1182-1-ND" H 1750 7650 50  0001 C CNN "Digi-Key PN"
 F 6 "https://www.digikey.com/product-detail/en/samsung-electro-mechanics/CL10A105KP8NNNC/1276-1182-1-ND/3889268" H 1750 7650 50  0001 C CNN "Digi-Key Page"
+F 7 "CL10A105KP8NNNC" H 1750 7650 50  0001 C CNN "part_num"
 	1    1750 7650
 	0    -1   1    0
@@
 F 5 "1276-1182-1-ND" H 1450 7750 50  0001 C CNN "Digi-Key PN"
 F 6 "https://www.digikey.com/product-detail/en/samsung-electro-mechanics/CL10A105KP8NNNC/1276-1182-1-ND/3889268" H 1450 7750 50  0001 C CNN "Digi-Key Page"
+F 7 "CL10A105KP8NNNC" H 1450 7750 50  0001 C CNN "part_num"
 	1    1450 7750
 	0    -1   1    0
@@
 F 5 "311-22.0HRCT-ND" H 2950 2350 50  0001 C CNN "Digi-Key PN"
 F 6 "https://www.digikey.com/product-detail/en/yageo/RC0603FR-0722RL/311-22.0HRCT-ND/730002" H 2950 2350 50  0001 C CNN "Digi-Key Page"
+F 7 "RC0603FR-0722RL" H 2950 2350 50  0001 C CNN "part_num"
 	1    2950 2350
 	0    1    1    0
@@
 F 5 "311-10.0KHRCT-ND" H 5500 3450 50  0001 C CNN "Digi-Key PN"
 F 6 "https://www.digikey.com/product-detail/en/yageo/RC0603FR-0710KL/311-10.0KHRCT-ND/729827" H 5500 3450 50  0001 C CNN "Digi-Key Page"
+F 7 "RC0603FR-0710KL" H 5500 3450 50  0001 C CNN "part_num"
 	1    5500 3450
 	0    1    1    0
@@
 F 5 "311-22.0HRCT-ND" H 2950 2450 50  0001 C CNN "Digi-Key PN"
 F 6 "https://www.digikey.com/product-detail/en/yageo/RC0603FR-0722RL/311-22.0HRCT-ND/730002" H 2950 2450 50  0001 C CNN "Digi-Key Page"
+F 7 "RC0603FR-0722RL" H 2950 2450 50  0001 C CNN "part_num"
 	1    2950 2450
 	0    1    1    0
@@
 F 5 "1276-1182-1-ND" H 3150 2650 50  0001 C CNN "Digi-Key PN"
 F 6 "https://www.digikey.com/product-detail/en/samsung-electro-mechanics/CL10A105KP8NNNC/1276-1182-1-ND/3889268" H 3150 2650 50  0001 C CNN "Digi-Key Page"
+F 7 "CL10A105KP8NNNC" H 3150 2650 50  0001 C CNN "part_num"
 	1    3150 2650
 	0    1    1    0
@@
 F 5 "1276-1005-1-ND" H 5950 4750 50  0001 C CNN "Digi-Key PN"
 F 6 "https://www.digikey.com/product-detail/en/samsung-electro-mechanics/CL10B104KO8NNNC/1276-1005-1-ND/3889091" H 5950 4750 50  0001 C CNN "Digi-Key Page"
+F 7 "CL10B104KO8NNNC" H 5950 4750 50  0001 C CNN "part_num"
 	1    5950 4750
 	-1   0    0    1
@@
 F 5 "296-14857-1-ND" H 5800 5600 50  0001 C CNN "Digi-Key PN"
 F 6 "https://www.digikey.com/product-detail/en/texas-instruments/SN74HC595DR/296-14857-1-ND/562567" H 5800 5600 50  0001 C CNN "Digi-Key Page"
+F 7 "SN74HC595DR" H 5800 5600 50  0001 C CNN "part_num"
 	1    5800 5600
 	1    0    0    -1
@@
 F 5 "311-10.0KHRCT-ND" H 1550 1100 50  0001 C CNN "Digi-Key PN"
 F 6 "https://www.digikey.com/product-detail/en/yageo/RC0603FR-0710KL/311-10.0KHRCT-ND/729827" H 1550 1100 50  0001 C CNN "Digi-Key Page"
+F 7 "RC0603FR-0710KL" H 1550 1100 50  0001 C CNN "part_num"
 	1    1550 1100
 	0    1    1    0
@@
 F 5 "CKN9112CT-ND" H 1550 1350 50  0001 C CNN "Digi-Key PN"
 F 6 "https://www.digikey.com/product-detail/en/c-k/PTS645SM43SMTR92-LFS/CKN9112CT-ND/1146934" H 1550 1350 50  0001 C CNN "Digi-Key Page"
+F 7 "PTS645SM43SMTR92 LFS" H 1550 1350 50  0001 C CNN "part_num"
 	1    1550 1350
 	1    0    0    -1
@@
 F 5 "311-1062-1-ND" H 750 2400 50  0001 C CNN "Digi-Key PN"
 F 6 "https://www.digikey.com/product-detail/en/yageo/CC0603JRNPO9BN220/311-1062-1-ND/302972" H 750 2400 50  0001 C CNN "Digi-Key Page"
+F 7 "CC0603JRNPO9BN220" H 750 2400 50  0001 C CNN "part_num"
 	1    750  2400
 	1    0    0    -1
@@
 F 5 "609-4613-1-ND" H 1900 2350 50  0001 C CNN "Digi-Key PN"
 F 6 "https://www.digikey.com/product-detail/en/amphenol-icc-fci/10118192-0001LF/609-4613-1-ND/2785378" H 1900 2350 50  0001 C CNN "Digi-Key Page"
+F 7 "10118192-0001LF" H 1900 2350 50  0001 C CNN "part_num"
 	1    1900 2350
 	1    0    0    -1
@@
 F 5 "311-1062-1-ND" H 1350 2400 50  0001 C CNN "Digi-Key PN"
 F 6 "https://www.digikey.com/product-detail/en/yageo/CC0603JRNPO9BN220/311-1062-1-ND/302972" H 1350 2400 50  0001 C CNN "Digi-Key Page"
+F 7 "CC0603JRNPO9BN220" H 1350 2400 50  0001 C CNN "part_num"
 	1    1350 2400
 	1    0    0    -1
@@
 F 5 "XC2103CT-ND" H 1050 2250 50  0001 C CNN "Digi-Key PN"
 F 6 "https://www.digikey.com/product-detail/en/ecs-inc/ECS-80-18-30-JGN-TR/XC2103CT-ND/5875587" H 1050 2250 50  0001 C CNN "Digi-Key Page"
+F 7 "ECS-80-18-30-JGN-TR" H 1050 2250 50  0001 C CNN "part_num"
 	1    1050 2250
 	1    0    0    -1
@@
 F 5 "https://www.digikey.com/product-detail/en/samsung-electro-mechanics/CL10A475KQ8NNNC/1276-1045-1-ND/3889131" H 3650 950 50  0001 C CNN "Digi-Key Page"
 F 6 "1276-1045-1-ND" H 3650 950 50  0001 C CNN "Digi-Key PN"
+F 7 "CL10A475KQ8NNNC" H 3650 950 50  0001 C CNN "part_num"
 	1    3650 950
 	0    -1   -1   0
@@
 F 5 "1727-3782-ND" H 1350 5300 50  0001 C CNN "Digi-Key PN"
 F 6 "https://www.digikey.com/product-detail/en/nexperia-usa-inc/74HC165D,652/1727-3782-ND/763577" H 1350 5300 50  0001 C CNN "Digi-Key Page"
+F 7 "74HC165D\\,652" H 1350 5300 50  0001 C CNN "part_num"
 	1    1350 5300
 	1    0    0    -1
@@
 F 5 "SML-D12U1WT86CT-ND" H 4850 2550 50  0001 C CNN "Digi-Key PN"
 F 6 "https://www.digikey.com/product-detail/en/rohm-semiconductor/SML-D12U1WT86/SML-D12U1WT86CT-ND/5843858" H 4850 2550 50  0001 C CNN "Digi-Key Page"
+F 7 "SML-D12U1WT86" H 4850 2550 50  0001 C CNN "part_num"
 	1    4850 2550
 	-1   0    0    1
@@
 F 5 "311-1.00KHRCT-ND" H 5200 2550 50  0001 C CNN "Digi-Key PN"
 F 6 "https://www.digikey.com/product-detail/en/yageo/RC0603FR-071KL/311-1.00KHRCT-ND/729790" H 5200 2550 50  0001 C CNN "Digi-Key Page"
+F 7 "RC0603FR-071KL" H 5200 2550 50  0001 C CNN "part_num"
 	1    5200 2550
 	0    -1   1    0
@@
 F 5 "ATMEGA32U4-AURCT-ND" H 4000 2850 50  0001 C CNN "Digi-Key PN"
 F 6 "https://www.digikey.com/product-detail/en/microchip-technology/ATMEGA32U4-AUR/ATMEGA32U4-AURCT-ND/3440960" H 4000 2850 50  0001 C CNN "Digi-Key Page"
+F 7 "ATMEGA32U4-AUR" H 4000 2850 50  0001 C CNN "part_num"
 	1    4000 2850
 	1    0    0    -1
