File: kicad/sheet_keymatrix.sch (KiCad schematic (older format))
At the start: 68 parts, among them SW10 SW_Push, SW12 SW_Push, SW14 SW_Push, SW15 SW_Push, SW16 SW_Push, SW17 SW_Push, SW18 SW_Push, SW19 SW_Push, SW21 SW_Push, SW22 SW_Push, SW23 SW_Push, SW24 SW_Push, SW25 SW_Push, SW26 SW_Push, SW28 SW_Push, SW3 SW_Push, SW30 SW_Push, SW31 SW_Push, SW32 SW_Push, SW33 SW_Push, SW34 SW_Push, SW35 SW_Push, SW36 SW_Push, SW37 SW_Push, SW38 SW_Push, SW39 SW_Push, SW4 SW_Push, SW40 SW_Push, SW41 SW_Push, SW42 SW_Push, SW43 SW_Push, SW44 SW_Push, SW45 SW_Push, SW46 SW_Push, SW47 SW_Push, SW5 SW_Push, SW50 SW_Push, SW51 SW_Push, SW52 SW_Push, SW53 SW_Push, SW54 SW_Push, SW55 SW_Push, SW58 SW_Push, SW59 SW_Push, SW6 SW_Push, SW60 SW_Push, SW61 SW_Push, SW62 SW_Push, SW63 SW_Push, SW7 SW_Push, SW8 SW_Push, SW9 SW_Push

Commit message: kicad: fix virtual component
Parts:
- D1, D2, D3, D4, D5, D6, D7, D8: part_num (none) -> TS4148C RZG
- R10, R11, R12, R5, R6, R7, R8, R9: part_num (none) -> RC0603FR-0710KL
Changed lines of the file:
@@
 F 5 "311-10.0KHRCT-ND" H 5850 4850 50  0001 C CNN "Digi-Key PN"
 F 6 "https://www.digikey.com/product-detail/en/yageo/RC0603FR-0710KL/311-10.0KHRCT-ND/729827" H 5850 4850 50  0001 C CNN "Digi-Key Page"
+F 7 "RC0603FR-0710KL" H 5850 4850 50  0001 C CNN "part_num"
 	1    5850 4850
 	0    1    1    0
@@
 F 5 "311-10.0KHRCT-ND" H 5850 4300 50  0001 C CNN "Digi-Key PN"
 F 6 "https://www.digikey.com/product-detail/en/yageo/RC0603FR-0710KL/311-10.0KHRCT-ND/729827" H 5850 4300 50  0001 C CNN "Digi-Key Page"
+F 7 "RC0603FR-0710KL" H 5850 4300 50  0001 C CNN "part_num"
 	1    5850 4300
 	0    1    1    0
@@
 F 5 "311-10.0KHRCT-ND" H 5850 3750 50  0001 C CNN "Digi-Key PN"
 F 6 "https://www.digikey.com/product-detail/en/yageo/RC0603FR-0710KL/311-10.0KHRCT-ND/729827" H 5850 3750 50  0001 C CNN "Digi-Key Page"
+F 7 "RC0603FR-0710KL" H 5850 3750 50  0001 C CNN "part_num"
 	1    5850 3750
 	0    1    1    0
@@
 F 5 "311-10.0KHRCT-ND" H 5850 3200 50  0001 C CNN "Digi-Key PN"
 F 6 "https://www.digikey.com/product-detail/en/yageo/RC0603FR-0710KL/311-10.0KHRCT-ND/729827" H 5850 3200 50  0001 C CNN "Digi-Key Page"
+F 7 "RC0603FR-0710KL" H 5850 3200 50  0001 C CNN "part_num"
 	1    5850 3200
 	0    1    1    0
@@
 F 5 "311-10.0KHRCT-ND" H 5850 2650 50  0001 C CNN "Digi-Key PN"
 F 6 "https://www.digikey.com/product-detail/en/yageo/RC0603FR-0710KL/311-10.0KHRCT-ND/729827" H 5850 2650 50  0001 C CNN "Digi-Key Page"
+F 7 "RC0603FR-0710KL" H 5850 2650 50  0001 C CNN "part_num"
 	1    5850 2650
 	0    1    1    0
@@
 F 5 "311-10.0KHRCT-ND" H 5850 2100 50  0001 C CNN "Digi-Key PN"
 F 6 "https://www.digikey.com/product-detail/en/yageo/RC0603FR-0710KL/311-10.0KHRCT-ND/729827" H 5850 2100 50  0001 C CNN "Digi-Key Page"
+F 7 "RC0603FR-0710KL" H 5850 2100 50  0001 C CNN "part_num"
 	1    5850 2100
 	0    1    1    0
@@
 F 5 "311-10.0KHRCT-ND" H 5850 1550 50  0001 C CNN "Digi-Key PN"
 F 6 "https://www.digikey.com/product-detail/en/yageo/RC0603FR-0710KL/311-10.0KHRCT-ND/729827" H 5850 1550 50  0001 C CNN "Digi-Key Page"
+F 7 "RC0603FR-0710KL" H 5850 1550 50  0001 C CNN "part_num"
 	1    5850 1550
 	0    1    1    0
@@
 F 5 "TS4148CRZGCT-ND" H 2900 1050 50  0001 C CNN "Digi-Key PN"
 F 6 "https://www.digikey.com/product-detail/en/taiwan-semiconductor-corporation/TS4148C-RZG/TS4148CRZGCT-ND/7359812" H 2900 1050 50  0001 C CNN "Digi-Key Page"
+F 7 "TS4148C RZG" H 2900 1050 50  0001 C CNN "part_num"
 	1    2900 1050
 	0    -1   -1   0
@@
 F 5 "TS4148CRZGCT-ND" H 3450 1050 50  0001 C CNN "Digi-Key PN"
 F 6 "https://www.digikey.com/product-detail/en/taiwan-semiconductor-corporation/TS4148C-RZG/TS4148CRZGCT-ND/7359812" H 3450 1050 50  0001 C CNN "Digi-Key Page"
+F 7 "TS4148C RZG" H 3450 1050 50  0001 C CNN "part_num"
 	1    3450 1050
 	0    -1   -1   0
@@
 F 5 "TS4148CRZGCT-ND" H 4550 1050 50  0001 C CNN "Digi-Key PN"
 F 6 "https://www.digikey.com/product-detail/en/taiwan-semiconductor-corporation/TS4148C-RZG/TS4148CRZGCT-ND/7359812" H 4550 1050 50  0001 C CNN "Digi-Key Page"
+F 7 "TS4148C RZG" H 4550 1050 50  0001 C CNN "part_num"
 	1    4550 1050
 	0    -1   -1   0
@@
 F 5 "TS4148CRZGCT-ND" H 5100 1050 50  0001 C CNN "Digi-Key PN"
 F 6 "https://www.digikey.com/product-detail/en/taiwan-semiconductor-corporation/TS4148C-RZG/TS4148CRZGCT-ND/7359812" H 5100 1050 50  0001 C CNN "Digi-Key Page"
+F 7 "TS4148C RZG" H 5100 1050 50  0001 C CNN "part_num"
 	1    5100 1050
 	0    -1   -1   0
@@
 F 5 "TS4148CRZGCT-ND" H 5650 1050 50  0001 C CNN "Digi-Key PN"
 F 6 "https://www.digikey.com/product-detail/en/taiwan-semiconductor-corporation/TS4148C-RZG/TS4148CRZGCT-ND/7359812" H 5650 1050 50  0001 C CNN "Digi-Key Page"
+F 7 "TS4148C RZG" H 5650 1050 50  0001 C CNN "part_num"
 	1    5650 1050
 	0    -1   -1   0
@@
 F 5 "TS4148CRZGCT-ND" H 2350 1050 50  0001 C CNN "Digi-Key PN"
 F 6 "https://www.digikey.com/product-detail/en/taiwan-semiconductor-corporation/TS4148C-RZG/TS4148CRZGCT-ND/7359812" H 2350 1050 50  0001 C CNN "Digi-Key Page"
+F 7 "TS4148C RZG" H 2350 1050 50  0001 C CNN "part_num"
 	1    2350 1050
 	0    -1   -1   0
@@
 F 5 "TS4148CRZGCT-ND" H 1800 1050 50  0001 C CNN "Digi-Key PN"
 F 6 "https://www.digikey.com/product-detail/en/taiwan-semiconductor-corporation/TS4148C-RZG/TS4148CRZGCT-ND/7359812" H 1800 1050 50  0001 C CNN "Digi-Key Page"
+F 7 "TS4148C RZG" H 1800 1050 50  0001 C CNN "part_num"
 	1    1800 1050
 	0    -1   -1   0
@@
 F 5 "TS4148CRZGCT-ND" H 4000 1050 50  0001 C CNN "Digi-Key PN"
 F 6 "https://www.digikey.com/product-detail/en/taiwan-semiconductor-corporation/TS4148C-RZG/TS4148CRZGCT-ND/7359812" H 4000 1050 50  0001 C CNN "Digi-Key Page"
+F 7 "TS4148C RZG" H 4000 1050 50  0001 C CNN "part_num"
 	1    4000 1050
 	0    -1   -1   0
@@
 F 5 "311-10.0KHRCT-ND" H 5850 5400 50  0001 C CNN "Digi-Key PN"
 F 6 "https://www.digikey.com/product-detail/en/yageo/RC0603FR-0710KL/311-10.0KHRCT-ND/729827" H 5850 5400 50  0001 C CNN "Digi-Key Page"
+F 7 "RC0603FR-0710KL" H 5850 5400 50  0001 C CNN "part_num"
 	1    5850 5400
 	0    1    1    0
